File: block.kicad_pcb (KiCad board)
At the start: 2 copper layers, 252.5 x 78.7 mm, 103 parts, among them J1 OLED, SW1 SW_PUSH, SW10 SW_PUSH, SW11 SW_PUSH, SW12 SW_PUSH, SW13 SW_PUSH, SW14 SW_PUSH, SW15 SW_PUSH, SW16 SW_PUSH, SW17 SW_PUSH, SW18 SW_PUSH, SW19 SW_PUSH, SW2 SW_PUSH, SW20 SW_PUSH, SW21 SW_PUSH, SW22 SW_PUSH, SW23 SW_PUSH, SW24 SW_PUSH, SW25 SW_PUSH, SW26 SW_PUSH, SW27 SW_PUSH, SW28 SW_PUSH, SW29 SW_PUSH, SW3 SW_PUSH, SW30 SW_PUSH, SW31 SW_PUSH, SW32 SW_PUSH, SW33 SW_PUSH, SW34 SW_PUSH, SW35 SW_PUSH, SW36 SW_PUSH, SW37 SW_PUSH, SW38 SW_PUSH, SW39 SW_PUSH, SW4 SW_PUSH, SW40 SW_PUSH, SW41 SW_PUSH, SW42 SW_PUSH, SW43 SW_PUSH, SW44 SW_PUSH, SW45 SW_PUSH, SW46 SW_PUSH, SW47 SW_PUSH, SW48 SW_PUSH, SW5 SW_PUSH, SW6 SW_PUSH, SW7 SW_PUSH, SW8 SW_PUSH, SW9 SW_PUSH, U1 ProMicro

Commit message: add ground fills
Routing:
- added copper zone on F.Cu, net GND
Changed lines of the file:
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@@
   (segment (start 37.55 80.719) (end 42.25 80.719) (width 0.25) (layer "B.Cu") (net 2))
   (segment (start 138.55 95.444) (end 137.099999 96.894001) (width 0.25) (layer "F.Cu") (net 3))
+  (segment (start 158.910918 95.619) (end 158.391647 96.138271) (width 0.25) (layer "F.Cu") (net 3))
   (segment (start 197.2 95.344) (end 205.459134 95.344) (width 0.25) (layer "F.Cu") (net 3))
   (segment (start 61.75 95.444) (end 70.009134 95.444) (width 0.25) (layer "F.Cu") (net 3))
+  (segment (start 157.152063 96.138271) (end 157.113792 96.1) (width 0.25) (layer "F.Cu") (net 3))
   (segment (start 254.8 95.344) (end 263.059134 95.344) (width 0.25) (layer "F.Cu") (net 3))
   (segment (start 186.259134 95.344) (end 187.709135 96.794001) (width 0.25) (layer "F.Cu") (net 3))
   (segment (start 79.499999 96.894001) (end 80.95 95.444) (width 0.25) (layer "F.Cu") (net 3))
-  (segment (start 158.210918 96.319) (end 143.650043 96.319) (width 0.25) (layer "F.Cu") (net 3))
-  (segment (start 158.910918 95.619) (end 158.210918 96.319) (width 0.25) (layer "F.Cu") (net 3))
   (segment (start 119.35 95.444) (end 117.899999 96.894001) (width 0.25) (layer "F.Cu") (net 3))
   (segment (start 106.426652 95.444) (end 100.15 95.444) (width 0.25) (layer "F.Cu") (net 3))
-  (segment (start 176.549999 96.794001) (end 166.625001 96.794001) (width 0.25) (layer "F.Cu") (net 3))
-  (segment (start 165.45 95.619) (end 158.910918 95.619) (width 0.25) (layer "F.Cu") (net 3))
   (segment (start 98.699999 96.894001) (end 100.15 95.444) (width 0.25) (layer "F.Cu") (net 3))
-  (segment (start 143.650043 96.319) (end 142.382314 95.051271) (width 0.25) (layer "F.Cu") (net 3))
   (segment (start 141.989585 95.444) (end 142.382314 95.051271) (width 0.25) (layer "F.Cu") (net 3))
   (segment (start 178 95.344) (end 186.259134 95.344) (width 0.25) (layer "F.Cu") (net 3))
-  (segment (start 166.625001 96.794001) (end 165.45 95.619) (width 0.25) (layer "F.Cu") (net 3))
   (segment (start 235.6 95.344) (end 243.859134 95.344) (width 0.25) (layer "F.Cu") (net 3))
   (segment (start 125.626652 95.444) (end 119.35 95.444) (width 0.25) (layer "F.Cu") (net 3))
+  (segment (start 165.45 95.619) (end 158.910918 95.619) (width 0.25) (layer "F.Cu") (net 3))
   (segment (start 107.876653 96.894001) (end 106.426652 95.444) (width 0.25) (layer "F.Cu") (net 3))
   (segment (start 137.099999 96.894001) (end 127.076653 96.894001) (width 0.25) (layer "F.Cu") (net 3))
@@
   (segment (start 187.709135 96.794001) (end 195.749999 96.794001) (width 0.25) (layer "F.Cu") (net 3))
   (segment (start 234.149999 96.794001) (end 235.6 95.344) (width 0.25) (layer "F.Cu") (net 3))
-  (segment (start 178 95.344) (end 176.549999 96.794001) (width 0.25) (layer "F.Cu") (net 3))
   (segment (start 214.949999 96.794001) (end 216.4 95.344) (width 0.25) (layer "F.Cu") (net 3))
   (segment (start 60.299999 96.894001) (end 61.75 95.444) (width 0.25) (layer "F.Cu") (net 3))
+  (segment (start 143.431043 96.1) (end 142.382314 95.051271) (width 0.25) (layer "F.Cu") (net 3))
   (segment (start 117.899999 96.894001) (end 107.876653 96.894001) (width 0.25) (layer "F.Cu") (net 3))
+  (segment (start 176.549999 96.794001) (end 166.625001 96.794001) (width 0.25) (layer "F.Cu") (net 3))
+  (segment (start 158.391647 96.138271) (end 157.152063 96.138271) (width 0.25) (layer "F.Cu") (net 3))
   (segment (start 224.659134 95.344) (end 226.109135 96.794001) (width 0.25) (layer "F.Cu") (net 3))
   (segment (start 52.259135 96.894001) (end 60.299999 96.894001) (width 0.25) (layer "F.Cu") (net 3))
@@
   (segment (start 127.076653 96.894001) (end 125.626652 95.444) (width 0.25) (layer "F.Cu") (net 3))
   (segment (start 272.549999 96.794001) (end 274 95.344) (width 0.25) (layer "F.Cu") (net 3))
+  (segment (start 157.113792 96.1) (end 143.431043 96.1) (width 0.25) (layer "F.Cu") (net 3))
   (segment (start 138.55 95.444) (end 141.989585 95.444) (width 0.25) (layer "F.Cu") (net 3))
   (segment (start 205.459134 95.344) (end 206.909135 96.794001) (width 0.25) (layer "F.Cu") (net 3))
@@
   (segment (start 206.909135 96.794001) (end 214.949999 96.794001) (width 0.25) (layer "F.Cu") (net 3))
   (segment (start 216.4 95.344) (end 224.659134 95.344) (width 0.25) (layer "F.Cu") (net 3))
+  (segment (start 178 95.344) (end 176.549999 96.794001) (width 0.25) (layer "F.Cu") (net 3))
   (segment (start 226.109135 96.794001) (end 234.149999 96.794001) (width 0.25) (layer "F.Cu") (net 3))
   (segment (start 50.809134 95.444) (end 52.259135 96.894001) (width 0.25) (layer "F.Cu") (net 3))
+  (segment (start 166.625001 96.794001) (end 165.45 95.619) (width 0.25) (layer "F.Cu") (net 3))
   (segment (start 40.092 88.939) (end 37.55 91.481) (width 0.25) (layer "B.Cu") (net 4))
   (segment (start 42.25 99.919) (end 42.55 100.219) (width 0.25) (layer "B.Cu") (net 4))
@@
   (segment (start 143.75 107.219) (end 143.75 81.178957) (width 0.25) (layer "B.Cu") (net 71))
   (segment (start 143.75 81.178957) (end 142.382314 79.811271) (width 0.25) (layer "B.Cu") (net 71))
+  (segment (start 149.931 106.019) (end 148.65038 106.019) (width 0.25) (layer "F.Cu") (net 72))
   (segment (start 148.65038 106.019) (end 148.65 106.01938) (width 0.25) (layer "F.Cu") (net 72))
   (segment (start 156.793585 85.7) (end 157.602314 84.891271) (width 0.25) (layer "F.Cu") (net 72))
   (segment (start 150.369 85.7) (end 156.793585 85.7) (width 0.25) (layer "F.Cu") (net 72))
   (segment (start 150.1345 85.9345) (end 150.369 85.7) (width 0.25) (layer "F.Cu") (net 72))
-  (segment (start 150.05 106.019) (end 148.65038 106.019) (width 0.25) (layer "F.Cu") (net 72))
-  (via (at 150.05 106.019) (size 0.8) (drill 0.4) (layers "F.Cu" "B.Cu") (net 72))
+  (via (at 149.931 106.019) (size 0.8) (drill 0.4) (layers "F.Cu" "B.Cu") (net 72))
   (via (at 150.1345 85.9345) (size 0.8) (drill 0.4) (layers "F.Cu" "B.Cu") (net 72))
-  (segment (start 150.1345 85.9345) (end 150.05 86.019) (width 0.25) (layer "B.Cu") (net 72))
-  (segment (start 150.05 86.019) (end 150.05 106.019) (width 0.25) (layer "B.Cu") (net 72))
+  (segment (start 149.931 106.019) (end 150.05 105.9) (width 0.25) (layer "B.Cu") (net 72))
+  (segment (start 150.05 105.9) (end 150.05 86.019) (width 0.25) (layer "B.Cu") (net 72))
+  (segment (start 150.05 86.019) (end 150.1345 85.9345) (width 0.25) (layer "B.Cu") (net 72))
   (segment (start 144.4745 83.8) (end 144.8745 83.4) (width 0.25) (layer "F.Cu") (net 73))
   (segment (start 146.05076 106.119) (end 146.15 106.01976) (width 0.25) (layer "F.Cu") (net 73))
@@
   (segment (start 153.65 80.619) (end 155.35 82.319) (width 0.25) (layer "B.Cu") (net 74))
   (segment (start 155.35 82.319) (end 155.35 102.619) (width 0.25) (layer "B.Cu") (net 74))
+  (zone (net 65) (net_name "GND") (layer "F.Cu") (hatch edge 0.508)
+    (connect_pads (clearance 0.508))
+    (min_thickness 0.254) (filled_areas_thickness no)
+    (fill yes (thermal_gap 0.508) (thermal_bridge_width 0.508) (island_removal_mode 2) (island_area_min 0))
+    (polygon
+      (pts
+        (xy 276.3 142.9)
+        (xy 23.7 143)
+        (xy 23.7 64.3)
+        (xy 276.3 64.2)
+      )
+    )
+  )
   (group "" (id 3bf397f5-7c11-4578-8f04-2d5dafcfda56)
     (members

Commit message: mounting holes
Parts:
- added ?: , kbd:LEGO_HOLE, F.Cu at (198.4, 84.3)
- added ?: , kbd:LEGO_HOLE, F.Cu at (256.1, 84.3)
- added ?: , kbd:LEGO_HOLE, F.Cu at (142.9, 109.8)
- added ?: , kbd:LEGO_HOLE, F.Cu at (256.1, 122.7)
- added ?: , kbd:LEGO_HOLE, F.Cu at (157.4, 109.8)
- added ?: , kbd:LEGO_HOLE, F.Cu at (198.4, 122.7)
- added M3: M2, kbd:LEGO_HOLE, F.Cu at (101.4, 84.4)
- added M4: M2, kbd:LEGO_HOLE, F.Cu at (101.4, 122.8)
- added M5: M2, kbd:LEGO_HOLE, F.Cu at (149.9, 115.0)
- added M6: M2, kbd:LEGO_HOLE, F.Cu at (149.9, 130.9)
- added MH1: M2, kbd:LEGO_HOLE, F.Cu at (43.8, 84.4)
- added MH2: M2, kbd:LEGO_HOLE, F.Cu at (43.8, 122.8)
- D1, D10, D11, D12, D13, D14, D15, D16, D17, D18, D19, D2, D20, D21, D22, D23, D24, D25, D26, D27, D28, D29, D3, D30, D31, D32, D33, D34, D35, D36, D37, D38, D39, D4, D40, D41, D42, D43, D44, D45, D46, D47, D48, D5, D6, D7, D8, D9: footprint kbd:D3_TH_SMD_v2 -> kbd:D3_SMD_v2; moved to B.Cu
- moved RSW1 8.15 mm to (149.8, 109.2), turned to 180 degrees
- moved D23 1.54 mm to (138.8, 118.0)
- moved D37 1.03 mm to (235.6, 79.0)
- moved D41 0.66 mm to (254.6, 78.5)
- moved D29 0.21 mm to (197.1, 78.1)
- moved D3 0.20 mm to (42.4, 116.4)
- moved D31 0.13 mm to (197.2, 116.2)
- moved D43 0.10 mm to (254.7, 116.3)
- moved D13 0.08 mm to (100.2, 78.1)
- moved D15 0.06 mm to (100.1, 116.5)
Routing:
- net row0: track 263.7 -> 313.4 mm, vias 1 -> 12
- net row2: track 262.4 -> 312.2 mm, vias 1 -> 12
- net row3: track 278.4 -> 327.6 mm, vias 1 -> 12
- net row1: track 245.4 -> 291.6 mm, vias 0 -> 12
- net reset: track 37.8 -> 52.8 mm
- net GND: track 55.2 -> 51.2 mm, vias 0 -> 1
- net col11: track 170.4 -> 173.8 mm
- net col2: track 145.4 -> 147.5 mm
- net col1: track 187.6 -> 189.5 mm
- net VCC: track 37.5 -> 36.1 mm
- net col10: track 149.7 -> 151.1 mm
- net Net-(D9-Pad1): track 17.2 -> 18.5 mm
- net col9: track 131.1 -> 132.4 mm
- net col3: track 126.7 -> 127.9 mm
- net col8: track 115.4 -> 116.5 mm
Other:
- board text added: "PCB design by bncpr"
- board text added: "block-kbd v1"

Commit message: add plates
Parts:
- MH10, MH7, MH8, MH9: renamed from ?; value (none) -> M2
- renumbered M3 to MH3, M4 to MH4, M5 to MH5, M6 to MH6
Routing:
- net row0: track 313.4 -> 264.4 mm
- net row3: track 327.6 -> 280.8 mm
- net row1: track 291.6 -> 245.5 mm
- net row2: track 312.2 -> 267.4 mm
